File: HARDWARE/Schematic/8051 Micocontroller.kicad_sch (KiCad schematic)
At the start: 31 parts, among them J3 Conn_01x04_Socket, U11 ADC082S051, U5 L293D, U6 P8051AH, U7 DM-OLED096-636, Y1 12MHz

Commit message: Validation files added and changes saved
Connections:
- net +5V: now also C13.2; no longer C13.1
- net at R10.1, U6.9 (RST): now also C13.1; no longer C13.2
Other:
- moved on the sheet: C13
Changed lines of the file:
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@@
 	(symbol
 		(lib_id "Device:C_Polarized")
-		(at 209.55 39.37 270)
+		(at 209.55 39.37 90)
 		(unit 1)
 		(exclude_from_sim no)
@@
 		(dnp no)
 		(property "Reference" "C13"
-			(at 207.772 32.766 90)
+			(at 211.074 33.02 90)
 			(effects
 				(font
@@
 		)
 		(property "Value" "10u"
-			(at 207.772 35.306 90)
+			(at 211.074 35.306 90)
 			(effects
 				(font
@@
 		)
 		(property "Footprint" "Capacitor_SMD:C_0805_2012Metric"
-			(at 205.74 40.3352 0)
+			(at 213.36 38.4048 0)
 			(effects
 				(font
